Commit message: Updated URDF to fix torso axes

File: backend/Testing/FullAssem11_24_23(1).urdf (robot description, URDF)
Before this commit: robot FullAssem11_24_23(1), 28 links, 27 joints
Links:
- link Belly: geometry collision mesh filename=package://FullAssem11_25_23/meshes/Belly.STL; visual mesh filename=package://FullAssem11_25_23/meshes/Belly.STL
- link BellyMotors: geometry collision mesh filename=package://FullAssem11_25_23/meshes/BellyMotors.STL; visual mesh filename=package://FullAssem11_25_23/meshes/BellyMotors.STL
- link Chest: geometry collision mesh filename=package://FullAssem11_25_23/meshes/Chest.STL; visual mesh filename=package://FullAssem11_25_23/meshes/Chest.STL
- link ChestMotors: geometry collision mesh filename=package://FullAssem11_25_23/meshes/ChestMotors.STL; visual mesh filename=package://FullAssem11_25_23/meshes/ChestMotors.STL
- link Head: geometry collision mesh filename=package://FullAssem11_25_23/meshes/Head.STL; visual mesh filename=package://FullAssem11_25_23/meshes/Head.STL
- link LeftBicep: geometry collision mesh filename=package://FullAssem11_25_23/meshes/LeftBicep.STL; visual mesh filename=package://FullAssem11_25_23/meshes/LeftBicep.STL
- link LeftFoot: geometry collision mesh filename=package://FullAssem11_25_23/meshes/LeftFoot.STL; visual mesh filename=package://FullAssem11_25_23/meshes/LeftFoot.STL
- link LeftForearm: geometry collision mesh filename=package://FullAssem11_25_23/meshes/LeftForearm.STL; visual mesh filename=package://FullAssem11_25_23/meshes/LeftForearm.STL
- link LeftHand: geometry collision mesh filename=package://FullAssem11_25_23/meshes/LeftHand.STL; visual mesh filename=package://FullAssem11_25_23/meshes/LeftHand.STL
- link LeftHip: geometry collision mesh filename=package://FullAssem11_25_23/meshes/LeftHip.STL; visual mesh filename=package://FullAssem11_25_23/meshes/LeftHip.STL
- link LeftHip2: geometry collision mesh filename=package://FullAssem11_25_23/meshes/LeftHip2.STL; visual mesh filename=package://FullAssem11_25_23/meshes/LeftHip2.STL
- link LeftShin: geometry collision mesh filename=package://FullAssem11_25_23/meshes/LeftShin.STL; visual mesh filename=package://FullAssem11_25_23/meshes/LeftShin.STL
- link LeftShoulder1: geometry collision mesh filename=package://FullAssem11_25_23/meshes/LeftShoulder1.STL; visual mesh filename=package://FullAssem11_25_23/meshes/LeftShoulder1.STL
- link LeftShoulder2: geometry collision mesh filename=package://FullAssem11_25_23/meshes/LeftShoulder2.STL; visual mesh filename=package://FullAssem11_25_23/meshes/LeftShoulder2.STL
- link LeftThigh: geometry collision mesh filename=package://FullAssem11_25_23/meshes/LeftThigh.STL; visual mesh filename=package://FullAssem11_25_23/meshes/LeftThigh.STL
- link Neck: geometry collision mesh filename=package://FullAssem11_25_23/meshes/Neck.STL; visual mesh filename=package://FullAssem11_25_23/meshes/Neck.STL
- link Pelvis: geometry collision mesh filename=package://FullAssem11_25_23/meshes/Pelvis.STL; visual mesh filename=package://FullAssem11_25_23/meshes/Pelvis.STL
- link RightBicep: geometry collision mesh filename=package://FullAssem11_25_23/meshes/RightBicep.STL; visual mesh filename=package://FullAssem11_25_23/meshes/RightBicep.STL
- link RightFoot: geometry collision mesh filename=package://FullAssem11_25_23/meshes/RightFoot.STL; visual mesh filename=package://FullAssem11_25_23/meshes/RightFoot.STL
- link RightForearm: geometry collision mesh filename=package://FullAssem11_25_23/meshes/RightForearm.STL; visual mesh filename=package://FullAssem11_25_23/meshes/RightForearm.STL
- link RightHand: geometry collision mesh filename=package://FullAssem11_25_23/meshes/RightHand.STL; visual mesh filename=package://FullAssem11_25_23/meshes/RightHand.STL
- link RightHip: geometry collision mesh filename=package://FullAssem11_25_23/meshes/RightHip.STL; visual mesh filename=package://FullAssem11_25_23/meshes/RightHip.STL
- link RightHip2: geometry collision mesh filename=package://FullAssem11_25_23/meshes/RightHip2.STL; visual mesh filename=package://FullAssem11_25_23/meshes/RightHip2.STL
- link RightShin: geometry collision mesh filename=package://FullAssem11_25_23/meshes/RightShin.STL; visual mesh filename=package://FullAssem11_25_23/meshes/RightShin.STL
- link RightShoulder1: geometry collision mesh filename=package://FullAssem11_25_23/meshes/RightShoulder1.STL; visual mesh filename=package://FullAssem11_25_23/meshes/RightShoulder1.STL
- link RightShoulder2: geometry collision mesh filename=package://FullAssem11_25_23/meshes/RightShoulder2.STL; visual mesh filename=package://FullAssem11_25_23/meshes/RightShoulder2.STL
- link RightThigh: geometry collision mesh filename=package://FullAssem11_25_23/meshes/RightThigh.STL; visual mesh filename=package://FullAssem11_25_23/meshes/RightThigh.STL
- link Torso: geometry collision mesh filename=package://FullAssem11_25_23/meshes/Torso.STL; visual mesh filename=package://FullAssem11_25_23/meshes/Torso.STL
Joints:
- joint HipsFront2Back: axis -1 0 0 -> 1 0 0
- joint HipsSide2Side: axis 0 0 -1 -> 0 0 1
- joint TorsoFront2Back: axis 0 -1 0 -> -1 0 0

Commit message: IKPY stuff n shi

File: backend/Testing/FullAssem11_24_23(1).urdf (robot description, URDF)
Before this commit: robot FullAssem11_25_23, 28 links, 27 joints
Joints:
- joint LeftAnkle: limit lower=0 upper=0 effort=0 velocity=0 -> (none)
- joint LeftKick: limit lower=0 upper=0 effort=0 velocity=0 -> (none)
- joint LeftKnee: limit lower=0 upper=0 effort=0 velocity=0 -> (none)
- joint LeftLegAbductor: limit lower=0 upper=0 effort=0 velocity=0 -> (none)
- joint LeftLegRotator: limit lower=0 upper=0 effort=0 velocity=0 -> (none)
- joint RightAnkle: limit lower=0 upper=0 effort=0 velocity=0 -> (none)
- joint RightKick: limit lower=0 upper=0 effort=0 velocity=0 -> (none)
- joint RightKnee: limit lower=0 upper=0 effort=0 velocity=0 -> (none)
- joint RightLegAbductor: limit lower=0 upper=0 effort=0 velocity=0 -> (none)
- joint RightLegRotator: limit lower=0 upper=0 effort=0 velocity=0 -> (none)
