Commit message: finally... movement

File: backend/Testing/robotChain.urdf (robot description, URDF)
Before this commit: robot FullAssem11_25_23, 28 links, 27 joints
Joints:
- joint LeftKnee: limit (none) -> lower=0 upper=6 effort=0 velocity=0
- joint RightKnee: limit (none) -> lower=-6 upper=0 effort=0 velocity=0

Commit message: Quintic sorta works, we're just trying to find out why we're unable to move the leg trajectories in to a negative task space position

File: backend/Testing/robotChain.urdf (robot description, URDF)
Before this commit: robot FullAssem11_25_23, 28 links, 27 joints
Joints:
- joint LeftKick: limit (none) -> lower=-4 upper=4 effort=0 velocity=0
- joint LeftKnee: limit (none) -> lower=0 upper=6 effort=0 velocity=0
- joint RightKick: limit (none) -> lower=-4 upper=4 effort=0 velocity=0
- joint RightKnee: limit (none) -> lower=-6 upper=0 effort=0 velocity=0

Commit message: doesn't work

File: backend/Testing/robotChain.urdf (robot description, URDF)
Before this commit: robot FullAssem11_25_23, 28 links, 27 joints
Joints:
- joint HeadNod: limit lower=0 upper=0 effort=0 velocity=0 -> (none)
- joint HipsFront2Back: limit lower=0 upper=0 effort=0 velocity=0 -> (none)
- joint HipsRotate: limit lower=0 upper=0 effort=0 velocity=0 -> (none)
- joint HipsSide2Side: limit lower=0 upper=0 effort=0 velocity=0 -> (none)
- joint LeftBicep: limit lower=0 upper=0 effort=0 velocity=0 -> (none)
- joint LeftElbow: limit lower=0 upper=0 effort=0 velocity=0 -> (none)
- joint LeftShoulderAbductor: limit lower=0 upper=0 effort=0 velocity=0 -> (none)
- joint LeftShoulderRotator: limit lower=0 upper=0 effort=0 velocity=0 -> (none)
- joint LeftWrist: limit lower=0 upper=0 effort=0 velocity=0 -> (none)
- joint Neck: limit lower=0 upper=0 effort=0 velocity=0 -> (none)
- joint RightBicep: limit lower=0 upper=0 effort=0 velocity=0 -> (none)
- joint RightElbow: limit lower=0 upper=0 effort=0 velocity=0 -> (none)
- joint RightShoulderAbductor: limit lower=0 upper=0 effort=0 velocity=0 -> (none)
- joint RightShoulderRotator: limit lower=0 upper=0 effort=0 velocity=0 -> (none)
- joint RightWrist: limit lower=0 upper=0 effort=0 velocity=0 -> (none)
- joint TorsoFront2Back: limit lower=0 upper=0 effort=0 velocity=0 -> (none)
- joint TorsoSide2Side: limit lower=0 upper=0 effort=0 velocity=0 -> (none)

Commit message: sim assisted walking works

File: backend/Testing/robotChain.urdf (robot description, URDF)
Before this commit: robot FullAssem11_25_23, 28 links, 27 joints
Joints:
- joint HeadNod: limit lower=0 upper=0 effort=0 velocity=0 -> (none)
- joint HipsRotate: limit lower=0 upper=0 effort=0 velocity=0 -> (none)
- joint LeftBicep: limit lower=0 upper=0 effort=0 velocity=0 -> (none)
- joint LeftElbow: limit lower=0 upper=0 effort=0 velocity=0 -> (none)
- joint LeftKick: limit lower=-4 upper=4 effort=0 velocity=0 -> (none)
- joint LeftKnee: axis 1 0 0 -> -1 0 0; limit lower=0 upper=6 effort=0 velocity=0 -> lower=-6 upper=0 effort=0 velocity=0
- joint LeftShoulderAbductor: limit lower=0 upper=0 effort=0 velocity=0 -> (none)
- joint LeftShoulderRotator: limit lower=0 upper=0 effort=0 velocity=0 -> (none)
- joint LeftWrist: limit lower=0 upper=0 effort=0 velocity=0 -> (none)
- joint Neck: limit lower=0 upper=0 effort=0 velocity=0 -> (none)
- joint RightBicep: limit lower=0 upper=0 effort=0 velocity=0 -> (none)
- joint RightElbow: limit lower=0 upper=0 effort=0 velocity=0 -> (none)
- joint RightKnee: axis -1 0 0 -> 1 0 0; limit lower=-6 upper=0 effort=0 velocity=0 -> lower=0 upper=6 effort=0 velocity=0
- joint RightShoulderAbductor: limit lower=0 upper=0 effort=0 velocity=0 -> (none)
- joint RightShoulderRotator: limit lower=0 upper=0 effort=0 velocity=0 -> (none)
- joint RightWrist: limit lower=0 upper=0 effort=0 velocity=0 -> (none)
- joint TorsoFront2Back: limit lower=0 upper=0 effort=0 velocity=0 -> (none)
- joint TorsoSide2Side: limit lower=0 upper=0 effort=0 velocity=0 -> (none)
